File: gps_backup.kicad_pcb (KiCad board)
At the start: 2 copper layers, 36.8 x 25.6 mm, 21 parts, among them J1 Conn_Coaxial, J2 Conn_01x04_Socket, J3 Conn_01x04_MountingPin, Q1 BSS138, Q2 BSS138, Q3 BSS138, Q4 BSS138, U1 MAX-M10S, U2 AP2112K-3.3

Commit message: layout, routing
Parts:
- moved C4 93.2 mm to (185.5, 104.0)
- moved C5 93.2 mm to (172.5, 110.5)
- moved J1 93.2 mm to (201.9, 110.8)
- moved Q3 93.2 mm to (181.4, 105.2)
- moved Q4 93.2 mm to (181.4, 108.7)
- moved R5 93.2 mm to (187.7, 94.4)
- moved C1 93.2 mm to (170.8, 100.2)
- moved C2 93.2 mm to (170.8, 98.4)
- moved C3 93.2 mm to (186.8, 98.7)
- moved J3 93.2 mm to (201.2, 94.2)
- moved Q1 93.2 mm to (192.9, 92.2)
- moved Q2 93.2 mm to (192.9, 95.8)
- moved R2 93.2 mm to (196.2, 96.5)
- moved R3 93.2 mm to (176.1, 89.3)
- moved R4 93.2 mm to (187.7, 91.0)
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Routing:
- net +3V3: track 39.2 -> 22.8 mm, vias 3 -> 2
Other:
- board size 36.8 x 25.6 mm -> 36.5 x 25.4 mm
